Commit message: Corrected Lidar Position in URDF

File: src/ppp_bot/description/lidar.xacro (robot description, xacro)
@@ -4,5 +4,5 @@
         <parent link="chassis"/>
         <child link="lidar_frame"/>
-        <origin xyz="0.1 0 0.19" rpy="0 0 0"/>
+        <origin xyz="0.15 0 0.15" rpy="0 0 0"/>
     </joint>
     <link name="lidar_frame">
